File: hardware/DOOR-8CH/kicad/DOOR-8CH.kicad_pcb (KiCad board)
At the start: 4 copper layers, 260 x 160 mm, 4 parts

Commit message: Place VNH channels and terminals on DOOR-8CH
Parts:
- added HS1A: M3.2 NPTH, TOP HEATSINK, MountingHole_3.2mm_M3, F.Cu at (24.0, 35.0)
- added HS1B: M3.2 NPTH, TOP HEATSINK, MountingHole_3.2mm_M3, F.Cu at (24.0, 61.0)
- added HS2A: M3.2 NPTH, TOP HEATSINK, MountingHole_3.2mm_M3, F.Cu at (54.0, 35.0)
- added HS2B: M3.2 NPTH, TOP HEATSINK, MountingHole_3.2mm_M3, F.Cu at (54.0, 61.0)
- added HS3A: M3.2 NPTH, TOP HEATSINK, MountingHole_3.2mm_M3, F.Cu at (84.0, 35.0)
- added HS3B: M3.2 NPTH, TOP HEATSINK, MountingHole_3.2mm_M3, F.Cu at (84.0, 61.0)
- added HS4A: M3.2 NPTH, TOP HEATSINK, MountingHole_3.2mm_M3, F.Cu at (114.0, 35.0)
- added HS4B: M3.2 NPTH, TOP HEATSINK, MountingHole_3.2mm_M3, F.Cu at (114.0, 61.0)
- added HS5A: M3.2 NPTH, TOP HEATSINK, MountingHole_3.2mm_M3, F.Cu at (146.0, 35.0)
- added HS5B: M3.2 NPTH, TOP HEATSINK, MountingHole_3.2mm_M3, F.Cu at (146.0, 61.0)
- added HS6A: M3.2 NPTH, TOP HEATSINK, MountingHole_3.2mm_M3, F.Cu at (176.0, 35.0)
- added HS6B: M3.2 NPTH, TOP HEATSINK, MountingHole_3.2mm_M3, F.Cu at (176.0, 61.0)
- added HS7A: M3.2 NPTH, TOP HEATSINK, MountingHole_3.2mm_M3, F.Cu at (206.0, 35.0)
- added HS7B: M3.2 NPTH, TOP HEATSINK, MountingHole_3.2mm_M3, F.Cu at (206.0, 61.0)
- added HS8A: M3.2 NPTH, TOP HEATSINK, MountingHole_3.2mm_M3, F.Cu at (236.0, 35.0)
- added HS8B: M3.2 NPTH, TOP HEATSINK, MountingHole_3.2mm_M3, F.Cu at (236.0, 61.0)
- added J1: FUSED_12V_CH1, TerminalBlock_Phoenix_MKDS-3-2-5.08_1x02_P5.08mm_Horizontal, F.Cu at (21.5, 76.0)
- added J10: ACTUATOR_CH2, TerminalBlock_Phoenix_MKDS-3-2-5.08_1x02_P5.08mm_Horizontal, F.Cu at (51.5, 91.0)
- added J11: ACTUATOR_CH3, TerminalBlock_Phoenix_MKDS-3-2-5.08_1x02_P5.08mm_Horizontal, F.Cu at (81.5, 91.0)
- added J12: ACTUATOR_CH4, TerminalBlock_Phoenix_MKDS-3-2-5.08_1x02_P5.08mm_Horizontal, F.Cu at (111.5, 91.0)
- added J13: ACTUATOR_CH5, TerminalBlock_Phoenix_MKDS-3-2-5.08_1x02_P5.08mm_Horizontal, F.Cu at (143.5, 91.0)
- added J14: ACTUATOR_CH6, TerminalBlock_Phoenix_MKDS-3-2-5.08_1x02_P5.08mm_Horizontal, F.Cu at (173.5, 91.0)
- added J15: ACTUATOR_CH7, TerminalBlock_Phoenix_MKDS-3-2-5.08_1x02_P5.08mm_Horizontal, F.Cu at (203.5, 91.0)
- added J16: ACTUATOR_CH8, TerminalBlock_Phoenix_MKDS-3-2-5.08_1x02_P5.08mm_Horizontal, F.Cu at (233.5, 91.0)
- added J2: FUSED_12V_CH2, TerminalBlock_Phoenix_MKDS-3-2-5.08_1x02_P5.08mm_Horizontal, F.Cu at (51.5, 76.0)
- added J3: FUSED_12V_CH3, TerminalBlock_Phoenix_MKDS-3-2-5.08_1x02_P5.08mm_Horizontal, F.Cu at (81.5, 76.0)
- added J4: FUSED_12V_CH4, TerminalBlock_Phoenix_MKDS-3-2-5.08_1x02_P5.08mm_Horizontal, F.Cu at (111.5, 76.0)
- added J5: FUSED_12V_CH5, TerminalBlock_Phoenix_MKDS-3-2-5.08_1x02_P5.08mm_Horizontal, F.Cu at (143.5, 76.0)
- added J6: FUSED_12V_CH6, TerminalBlock_Phoenix_MKDS-3-2-5.08_1x02_P5.08mm_Horizontal, F.Cu at (173.5, 76.0)
- added J7: FUSED_12V_CH7, TerminalBlock_Phoenix_MKDS-3-2-5.08_1x02_P5.08mm_Horizontal, F.Cu at (203.5, 76.0)
- added J8: FUSED_12V_CH8, TerminalBlock_Phoenix_MKDS-3-2-5.08_1x02_P5.08mm_Horizontal, F.Cu at (233.5, 76.0)
- added J9: ACTUATOR_CH1, TerminalBlock_Phoenix_MKDS-3-2-5.08_1x02_P5.08mm_Horizontal, F.Cu at (21.5, 91.0)
- added JSTM1A: STM32_SLOT_S1_LEFT, PinSocket_1x15_P2.54mm_Vertical, F.Cu at (24.8, 108.0)
- added JSTM1B: STM32_SLOT_S1_RIGHT, PinSocket_1x15_P2.54mm_Vertical, F.Cu at (45.2, 108.0)
- added JSTM2A: STM32_SLOT_S2_LEFT, PinSocket_1x15_P2.54mm_Vertical, F.Cu at (84.8, 108.0)
- added JSTM2B: STM32_SLOT_S2_RIGHT, PinSocket_1x15_P2.54mm_Vertical, F.Cu at (105.2, 108.0)
- added JSTM3A: STM32_SLOT_S3_LEFT, PinSocket_1x15_P2.54mm_Vertical, F.Cu at (144.8, 108.0)
- added JSTM3B: STM32_SLOT_S3_RIGHT, PinSocket_1x15_P2.54mm_Vertical, F.Cu at (165.2, 108.0)
- added JSTM4A: STM32_SLOT_S4_LEFT, PinSocket_1x15_P2.54mm_Vertical, F.Cu at (204.8, 108.0)
- added JSTM4B: STM32_SLOT_S4_RIGHT, PinSocket_1x15_P2.54mm_Vertical, F.Cu at (225.2, 108.0)
- added U1: VNH5019A-E, ST_MultiPowerSO-30, F.Cu at (24.0, 48.0)
- added U2: VNH5019A-E, ST_MultiPowerSO-30, F.Cu at (54.0, 48.0)
- added U3: VNH5019A-E, ST_MultiPowerSO-30, F.Cu at (84.0, 48.0)
- added U4: VNH5019A-E, ST_MultiPowerSO-30, F.Cu at (114.0, 48.0)
- added U5: VNH5019A-E, ST_MultiPowerSO-30, F.Cu at (146.0, 48.0)
- added U6: VNH5019A-E, ST_MultiPowerSO-30, F.Cu at (176.0, 48.0)
- added U7: VNH5019A-E, ST_MultiPowerSO-30, F.Cu at (206.0, 48.0)
- added U8: VNH5019A-E, ST_MultiPowerSO-30, F.Cu at (236.0, 48.0)

Commit message: Add control-module sockets to DOOR-8CH placement
Parts:
- added J101: SN65HVD230_MASTER_CAN, PinSocket_1x06_P2.54mm_Vertical, F.Cu at (18.0, 112.0)
- added J102: SN65HVD230_ESP_CAN_OPTION, PinSocket_1x06_P2.54mm_Vertical, F.Cu at (38.0, 112.0)
- added J103: CC1101_433MHZ, PinSocket_2x04_P2.54mm_Vertical, F.Cu at (58.0, 112.0)
- added J104: REEDS_3V3_GND, PinSocket_1x05_P2.54mm_Vertical, F.Cu at (78.0, 112.0)
- added J105: SWD_S1, PinSocket_1x06_P2.54mm_Vertical, F.Cu at (92.0, 112.0)

Commit message: Correct DOOR-8CH placement from module photos
Parts:
- removed J101: SN65HVD230_MASTER_CAN, PinSocket_1x06_P2.54mm_Vertical
- removed J102: SN65HVD230_ESP_CAN_OPTION, PinSocket_1x06_P2.54mm_Vertical
- removed J103: CC1101_433MHZ, PinSocket_2x04_P2.54mm_Vertical
- removed JSTM1A: STM32_SLOT_S1_LEFT, PinSocket_1x15_P2.54mm_Vertical
- removed JSTM1B: STM32_SLOT_S1_RIGHT, PinSocket_1x15_P2.54mm_Vertical
- removed JSTM2A: STM32_SLOT_S2_LEFT, PinSocket_1x15_P2.54mm_Vertical
- removed JSTM2B: STM32_SLOT_S2_RIGHT, PinSocket_1x15_P2.54mm_Vertical
- removed JSTM3A: STM32_SLOT_S3_LEFT, PinSocket_1x15_P2.54mm_Vertical
- removed JSTM3B: STM32_SLOT_S3_RIGHT, PinSocket_1x15_P2.54mm_Vertical
- removed JSTM4A: STM32_SLOT_S4_LEFT, PinSocket_1x15_P2.54mm_Vertical
- removed JSTM4B: STM32_SLOT_S4_RIGHT, PinSocket_1x15_P2.54mm_Vertical
- added CAN1: SN65HVD230_MASTER_CAN, SN65HVD230_Module_14.5x16.1mm_1x06, F.Cu at (63.0, 142.0)
- added CAN2: SN65HVD230_ESP_CAN_OPTION, SN65HVD230_Module_14.5x16.1mm_1x06, F.Cu at (123.0, 142.0)
- added CAP1: CAP1188_SPI, CAP1188_Adafruit1602_Module_2x13, F.Cu at (239.0, 70.0)
- added ESP1: ESP32_S3_DEVKITC_DOUBLE_DOOR_ONLY, ESP32-S3-DevKitC, F.Cu at (8.00, 105.0)
- added MOD1: STM32F103C8T6_MINI_SLOT_S1, STM32F103C8T6_Mini_CH340_4x10, F.Cu at (55.2, 153.0)
- added MOD2: STM32F103C8T6_MINI_SLOT_S2, STM32F103C8T6_Mini_CH340_4x10, F.Cu at (115.2, 153.0)
- added MOD3: STM32F103C8T6_MINI_SLOT_S3, STM32F103C8T6_Mini_CH340_4x10, F.Cu at (175.2, 153.0)
- added MOD4: STM32F103C8T6_MINI_SLOT_S4, STM32F103C8T6_Mini_CH340_4x10, F.Cu at (235.2, 153.0)
- added RF1: CC1101_433MHZ, CC1101_433MHz_Module_28x15mm_2x04, F.Cu at (31.0, 130.0)
- H1, H2, H3, H4: value M3.2 NPTH -> M3.2_NPTH; footprint DOOR-8CH:MountingHole_M3_2_NPTH -> MountingHole_M3_2_NPTH
- moved J104 175.2 mm to (253.0, 120.0), turned to -90 degrees
- moved J105 163.4 mm to (253.0, 140.0), turned to -90 degrees
- moved J10 83.3 mm to (58.0, 8.00)
- moved J11 83.3 mm to (88.0, 8.00)
- moved J12 83.3 mm to (118.0, 8.00)
- moved J13 83.3 mm to (150.0, 8.00)
- moved J14 83.3 mm to (180.0, 8.00)
- moved J15 83.3 mm to (210.0, 8.00)
- moved J16 83.3 mm to (240.0, 8.00)
- moved J9 83.3 mm to (28.0, 8.00)
- moved H2 70.5 mm to (230.0, 75.0)
- moved J1 68.3 mm to (15.0, 8.00)
- moved J2 68.3 mm to (45.0, 8.00)
- moved J3 68.3 mm to (75.0, 8.00)
- moved J4 68.3 mm to (105.0, 8.00)
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Other:
- board text removed: "4 LAYERS / 2 OZ OUTER COPPER / DO NOT FABRICATE YET"
- board text removed: "ACTUATOR POWER / VNH5019A-E"
- board text removed: "DOOR-8CH v0.1 - PRELIMINARY PLACEMENT"
- board text removed: "ESP32-S3 / CC1101 / ESP-CAN DOUBLE DOOR ONLY"
- board text removed: "LOGIC 5V IN CAN IN REEDS CAP1188 SWD"
- board text removed: "LOW VOLTAGE AND CONTROL"
- board text removed: "S1 MASTER / CAN / CAP1188 / REEDS / EEPROM"
- board text removed: "S1 STM32 2 x VNH"
- board text removed: "S2 STM32 2 x VNH"
- board text removed: "S3 STM32 2 x VNH"
- board text removed: "S4 STM32 2 x VNH"

Commit message: Add CAP1188 configuration and onboard power layout
Parts:
- removed J104: REEDS_3V3_GND, PinSocket_1x05_P2.54mm_Vertical
- removed J105: SWD_S1, PinSocket_1x06_P2.54mm_Vertical
- added C230: 470UF_50V, CP_Radial_D10.0mm_P5.00mm, F.Cu at (68.0, 68.0)
- added C231: 1UF_50V, C_1206_3216Metric, F.Cu at (81.0, 66.0)
- added C232: 100NF_50V, C_0603_1608Metric, F.Cu at (87.0, 66.0)
- added C233: 220UF_10V, CP_Radial_D8.0mm_P3.50mm, F.Cu at (128.0, 68.0)
- added C234: 10UF_10V, C_1206_3216Metric, F.Cu at (140.0, 66.0)
- added C235: 100NF_16V, C_0603_1608Metric, F.Cu at (146.0, 66.0)
- added D230: SS54_REVERSE_POLARITY, D_SMB, F.Cu at (42.0, 67.0)
- added D231: SMBJ16A_TVS, D_SMB, F.Cu at (54.0, 67.0)
- added DC1: MP1584_FIXED_5V, MP1584_Fixed5V_Module_22.3x17mm, F.Cu at (100.0, 65.0)
- added F230: 1A_SLOW_5X20, Fuseholder_Clip-5x20mm_Bel_FC-203-22_Lateral_P17.80x5.00mm_D1.17mm_Horizontal, F.Cu at (17.0, 67.0)
- added J201: REED_A_OPEN_3V3_SIG_GND, TerminalBlock_Phoenix_PT-1,5-3-3.5-H_1x03_P3.50mm_Horizontal, F.Cu at (254.7, 91.7)
- added J202: REED_A_CLOSED_3V3_SIG_GND, TerminalBlock_Phoenix_PT-1,5-3-3.5-H_1x03_P3.50mm_Horizontal, F.Cu at (254.7, 103.7)
- added J203: REED_A_IN_PLACE_3V3_SIG_GND, TerminalBlock_Phoenix_PT-1,5-3-3.5-H_1x03_P3.50mm_Horizontal, F.Cu at (254.7, 115.8)
- added J204: REED_B_OPEN_3V3_SIG_GND, TerminalBlock_Phoenix_PT-1,5-3-3.5-H_1x03_P3.50mm_Horizontal, F.Cu at (254.7, 127.8)
- added J205: REED_B_CLOSED_3V3_SIG_GND, TerminalBlock_Phoenix_PT-1,5-3-3.5-H_1x03_P3.50mm_Horizontal, F.Cu at (254.7, 139.9)
- added J206: REED_B_IN_PLACE_3V3_SIG_GND, TerminalBlock_Phoenix_PT-1,5-3-3.5-H_1x03_P3.50mm_Horizontal, F.Cu at (254.7, 151.9)
- added J211: CAP_CS1_GND, TerminalBlock_Phoenix_PT-1,5-2-3.5-H_1x02_P3.50mm_Horizontal, F.Cu at (254.7, 19.8)
- added J212: CAP_CS2_GND, TerminalBlock_Phoenix_PT-1,5-2-3.5-H_1x02_P3.50mm_Horizontal, F.Cu at (254.7, 28.3)
- added J213: CAP_CS3_GND, TerminalBlock_Phoenix_PT-1,5-2-3.5-H_1x02_P3.50mm_Horizontal, F.Cu at (254.7, 36.9)
- added J214: CAP_CS4_GND, TerminalBlock_Phoenix_PT-1,5-2-3.5-H_1x02_P3.50mm_Horizontal, F.Cu at (254.7, 45.4)
- added J215: CAP_CS5_GND, TerminalBlock_Phoenix_PT-1,5-2-3.5-H_1x02_P3.50mm_Horizontal, F.Cu at (254.7, 54.0)
- added J216: CAP_CS6_GND, TerminalBlock_Phoenix_PT-1,5-2-3.5-H_1x02_P3.50mm_Horizontal, F.Cu at (254.7, 62.5)
- added J217: CAP_CS7_GND, TerminalBlock_Phoenix_PT-1,5-2-3.5-H_1x02_P3.50mm_Horizontal, F.Cu at (254.7, 71.1)
- added J218: CAP_CS8_GND, TerminalBlock_Phoenix_PT-1,5-2-3.5-H_1x02_P3.50mm_Horizontal, F.Cu at (254.7, 79.6)
- added J220: SWD_S1_3V3_DIO_CLK_NRST_GND, PinHeader_1x05_P2.54mm_Vertical, F.Cu at (244.0, 128.0)
- added J230: LOGIC_12V_GND, TerminalBlock_Phoenix_PT-1,5-2-3.5-H_1x02_P3.50mm_Horizontal, F.Cu at (5.00, 60.0)
- added R201: 1K_CAP_INPUT, R_0603_1608Metric, F.Cu at (247.0, 18.0)
- added R202: 1K_CAP_INPUT, R_0603_1608Metric, F.Cu at (247.0, 26.6)
- added R203: 1K_CAP_INPUT, R_0603_1608Metric, F.Cu at (247.0, 35.1)
- added R204: 1K_CAP_INPUT, R_0603_1608Metric, F.Cu at (247.0, 43.7)
- added R205: 1K_CAP_INPUT, R_0603_1608Metric, F.Cu at (247.0, 52.2)
- added R206: 1K_CAP_INPUT, R_0603_1608Metric, F.Cu at (247.0, 60.8)
- added R207: 1K_CAP_INPUT, R_0603_1608Metric, F.Cu at (247.0, 69.3)
- added R208: 1K_CAP_INPUT, R_0603_1608Metric, F.Cu at (247.0, 77.9)
- added R209: 10K_CAP_RESET_PULLDOWN, R_0603_1608Metric, F.Cu at (215.0, 82.0)
- added R210: 10K_CAP_IRQ_PULLUP, R_0603_1608Metric, F.Cu at (215.0, 88.0)
- moved H2 22.0 mm to (208.0, 75.0)
- moved CAP1 21.5 mm to (220.0, 80.0)
- moved H4 9.00 mm to (243.0, 152.0)

Commit message: Add DOOR-8CH VNH electrical placement
Parts:
- added C1101: 470uF 35V LOW_ESR, CP_Radial_D10.0mm_P5.00mm, F.Cu at (16.0, 74.0)
- added C1102: 100nF 50V X7R VCC, C_0603_1608Metric, F.Cu at (34.0, 68.0)
- added C1103: 100nF ADC_FILTER, C_0603_1608Metric, F.Cu at (34.0, 72.0)
- added C1201: 470uF 35V LOW_ESR, CP_Radial_D10.0mm_P5.00mm, F.Cu at (46.0, 74.0)
- added C1202: 100nF 50V X7R VCC, C_0603_1608Metric, F.Cu at (64.0, 68.0)
- added C1203: 100nF ADC_FILTER, C_0603_1608Metric, F.Cu at (64.0, 72.0)
- added C1301: 470uF 35V LOW_ESR, CP_Radial_D10.0mm_P5.00mm, F.Cu at (76.0, 76.0)
- added C1302: 100nF 50V X7R VCC, C_0603_1608Metric, F.Cu at (94.0, 68.0)
- added C1303: 100nF ADC_FILTER, C_0603_1608Metric, F.Cu at (94.0, 72.0)
- added C1401: 470uF 35V LOW_ESR, CP_Radial_D10.0mm_P5.00mm, F.Cu at (106.0, 76.0)
- added C1402: 100nF 50V X7R VCC, C_0603_1608Metric, F.Cu at (124.0, 68.0)
- added C1403: 100nF ADC_FILTER, C_0603_1608Metric, F.Cu at (124.0, 72.0)
- added C1501: 470uF 35V LOW_ESR, CP_Radial_D10.0mm_P5.00mm, F.Cu at (138.0, 76.0)
- added C1502: 100nF 50V X7R VCC, C_0603_1608Metric, F.Cu at (156.0, 68.0)
- added C1503: 100nF ADC_FILTER, C_0603_1608Metric, F.Cu at (156.0, 72.0)
- added C1601: 470uF 35V LOW_ESR, CP_Radial_D10.0mm_P5.00mm, F.Cu at (168.0, 76.0)
- added C1602: 100nF 50V X7R VCC, C_0603_1608Metric, F.Cu at (186.0, 68.0)
- added C1603: 100nF ADC_FILTER, C_0603_1608Metric, F.Cu at (186.0, 72.0)
- added C1701: 470uF 35V LOW_ESR, CP_Radial_D10.0mm_P5.00mm, F.Cu at (191.0, 74.0)
- added C1702: 100nF 50V X7R VCC, C_0603_1608Metric, F.Cu at (214.0, 78.0)
- added C1703: 100nF ADC_FILTER, C_0603_1608Metric, F.Cu at (208.0, 82.0)
- added C1801: 470uF 35V LOW_ESR, CP_Radial_D10.0mm_P5.00mm, F.Cu at (218.0, 70.0)
- added C1802: 100nF 50V X7R VCC, C_0603_1608Metric, F.Cu at (244.0, 74.0)
- added C1803: 100nF ADC_FILTER, C_0603_1608Metric, F.Cu at (244.0, 78.0)
- added D1101: BAT54S ADC_CLAMP, SOT-23, F.Cu at (29.0, 72.0)
- added D1201: BAT54S ADC_CLAMP, SOT-23, F.Cu at (59.0, 72.0)
- added D1301: BAT54S ADC_CLAMP, SOT-23, F.Cu at (89.0, 72.0)
- added D1401: BAT54S ADC_CLAMP, SOT-23, F.Cu at (119.0, 72.0)
- added D1501: BAT54S ADC_CLAMP, SOT-23, F.Cu at (151.0, 72.0)
- added D1601: BAT54S ADC_CLAMP, SOT-23, F.Cu at (181.0, 72.0)
- added D1701: BAT54S ADC_CLAMP, SOT-23, F.Cu at (210.0, 78.0)
- added D1801: BAT54S ADC_CLAMP, SOT-23, F.Cu at (240.0, 76.0)
- added R1101: 100R INA_SER, R_0603_1608Metric, F.Cu at (16.0, 64.0)
- added R1102: 100R INB_SER, R_0603_1608Metric, F.Cu at (20.0, 64.0)
- added R1103: 100R PWM_SER, R_0603_1608Metric, F.Cu at (24.0, 64.0)
- added R1104: 10K INA_PULLDOWN, R_0603_1608Metric, F.Cu at (28.0, 64.0)
- added R1105: 10K INB_PULLDOWN, R_0603_1608Metric, F.Cu at (32.0, 64.0)
- added R1106: 10K PWM_PULLDOWN, R_0603_1608Metric, F.Cu at (36.0, 64.0)
- added R1107: 4K7 DIAG_PULLUP, R_0603_1608Metric, F.Cu at (18.0, 68.0)
- added R1108: 10K CS_DIS_PULLDOWN, R_0603_1608Metric, F.Cu at (22.0, 68.0)
- added R1109: 1K 1% CS_LOAD, R_0603_1608Metric, F.Cu at (26.0, 68.0)
- added R1110: 10K ADC_SERIES, R_0603_1608Metric, F.Cu at (30.0, 68.0)
- added R1201: 100R INA_SER, R_0603_1608Metric, F.Cu at (46.0, 64.0)
- added R1202: 100R INB_SER, R_0603_1608Metric, F.Cu at (50.0, 64.0)
- added R1203: 100R PWM_SER, R_0603_1608Metric, F.Cu at (54.0, 64.0)
- added R1204: 10K INA_PULLDOWN, R_0603_1608Metric, F.Cu at (58.0, 64.0)
- added R1205: 10K INB_PULLDOWN, R_0603_1608Metric, F.Cu at (62.0, 64.0)
- added R1206: 10K PWM_PULLDOWN, R_0603_1608Metric, F.Cu at (66.0, 64.0)
- added R1207: 4K7 DIAG_PULLUP, R_0603_1608Metric, F.Cu at (48.0, 68.0)
- added R1208: 10K CS_DIS_PULLDOWN, R_0603_1608Metric, F.Cu at (52.0, 68.0)
- added R1209: 1K 1% CS_LOAD, R_0603_1608Metric, F.Cu at (56.0, 68.0)
- added R1210: 10K ADC_SERIES, R_0603_1608Metric, F.Cu at (60.0, 68.0)
- added R1301: 100R INA_SER, R_0603_1608Metric, F.Cu at (76.0, 64.0)
- added R1302: 100R INB_SER, R_0603_1608Metric, F.Cu at (80.0, 64.0)
- added R1303: 100R PWM_SER, R_0603_1608Metric, F.Cu at (84.0, 64.0)
- added R1304: 10K INA_PULLDOWN, R_0603_1608Metric, F.Cu at (88.0, 64.0)
- added R1305: 10K INB_PULLDOWN, R_0603_1608Metric, F.Cu at (92.0, 64.0)
- added R1306: 10K PWM_PULLDOWN, R_0603_1608Metric, F.Cu at (96.0, 64.0)
- added R1307: 4K7 DIAG_PULLUP, R_0603_1608Metric, F.Cu at (78.0, 68.0)
- added R1308: 10K CS_DIS_PULLDOWN, R_0603_1608Metric, F.Cu at (82.0, 68.0)
- added R1309: 1K 1% CS_LOAD, R_0603_1608Metric, F.Cu at (86.0, 68.0)
- added R1310: 10K ADC_SERIES, R_0603_1608Metric, F.Cu at (90.0, 68.0)
- added R1401: 100R INA_SER, R_0603_1608Metric, F.Cu at (106.0, 64.0)
- added R1402: 100R INB_SER, R_0603_1608Metric, F.Cu at (110.0, 64.0)
- added R1403: 100R PWM_SER, R_0603_1608Metric, F.Cu at (114.0, 64.0)
- added R1404: 10K INA_PULLDOWN, R_0603_1608Metric, F.Cu at (118.0, 64.0)
- added R1405: 10K INB_PULLDOWN, R_0603_1608Metric, F.Cu at (122.0, 64.0)
- added R1406: 10K PWM_PULLDOWN, R_0603_1608Metric, F.Cu at (126.0, 64.0)
- added R1407: 4K7 DIAG_PULLUP, R_0603_1608Metric, F.Cu at (108.0, 68.0)
- added R1408: 10K CS_DIS_PULLDOWN, R_0603_1608Metric, F.Cu at (112.0, 68.0)
- added R1409: 1K 1% CS_LOAD, R_0603_1608Metric, F.Cu at (116.0, 68.0)
- added R1410: 10K ADC_SERIES, R_0603_1608Metric, F.Cu at (120.0, 68.0)
- added R1501: 100R INA_SER, R_0603_1608Metric, F.Cu at (138.0, 64.0)
- added R1502: 100R INB_SER, R_0603_1608Metric, F.Cu at (142.0, 64.0)
- added R1503: 100R PWM_SER, R_0603_1608Metric, F.Cu at (146.0, 64.0)
- added R1504: 10K INA_PULLDOWN, R_0603_1608Metric, F.Cu at (150.0, 64.0)
- added R1505: 10K INB_PULLDOWN, R_0603_1608Metric, F.Cu at (154.0, 64.0)
- added R1506: 10K PWM_PULLDOWN, R_0603_1608Metric, F.Cu at (158.0, 64.0)
- added R1507: 4K7 DIAG_PULLUP, R_0603_1608Metric, F.Cu at (140.0, 68.0)
- added R1508: 10K CS_DIS_PULLDOWN, R_0603_1608Metric, F.Cu at (144.0, 68.0)
- added R1509: 1K 1% CS_LOAD, R_0603_1608Metric, F.Cu at (148.0, 68.0)
- added R1510: 10K ADC_SERIES, R_0603_1608Metric, F.Cu at (152.0, 68.0)
- added R1601: 100R INA_SER, R_0603_1608Metric, F.Cu at (168.0, 64.0)
- added R1602: 100R INB_SER, R_0603_1608Metric, F.Cu at (172.0, 64.0)
- added R1603: 100R PWM_SER, R_0603_1608Metric, F.Cu at (176.0, 64.0)
- added R1604: 10K INA_PULLDOWN, R_0603_1608Metric, F.Cu at (180.0, 64.0)
- added R1605: 10K INB_PULLDOWN, R_0603_1608Metric, F.Cu at (184.0, 64.0)
- added R1606: 10K PWM_PULLDOWN, R_0603_1608Metric, F.Cu at (188.0, 64.0)
- added R1607: 4K7 DIAG_PULLUP, R_0603_1608Metric, F.Cu at (170.0, 68.0)
- added R1608: 10K CS_DIS_PULLDOWN, R_0603_1608Metric, F.Cu at (174.0, 68.0)
- added R1609: 1K 1% CS_LOAD, R_0603_1608Metric, F.Cu at (178.0, 68.0)
- added R1610: 10K ADC_SERIES, R_0603_1608Metric, F.Cu at (182.0, 68.0)
- added R1701: 100R INA_SER, R_0603_1608Metric, F.Cu at (198.0, 64.0)
- added R1702: 100R INB_SER, R_0603_1608Metric, F.Cu at (202.0, 64.0)
- added R1703: 100R PWM_SER, R_0603_1608Metric, F.Cu at (206.0, 64.0)
- added R1704: 10K INA_PULLDOWN, R_0603_1608Metric, F.Cu at (210.0, 64.0)
- added R1705: 10K INB_PULLDOWN, R_0603_1608Metric, F.Cu at (214.0, 64.0)
- added R1706: 10K PWM_PULLDOWN, R_0603_1608Metric, F.Cu at (218.0, 64.0)
- added R1707: 4K7 DIAG_PULLUP, R_0603_1608Metric, F.Cu at (200.0, 68.0)
- added R1708: 10K CS_DIS_PULLDOWN, R_0603_1608Metric, F.Cu at (204.0, 68.0)
- added R1709: 1K 1% CS_LOAD, R_0603_1608Metric, F.Cu at (208.0, 68.0)
- added R1710: 10K ADC_SERIES, R_0603_1608Metric, F.Cu at (212.0, 68.0)
- added R1801: 100R INA_SER, R_0603_1608Metric, F.Cu at (228.0, 64.0)
- added R1802: 100R INB_SER, R_0603_1608Metric, F.Cu at (232.0, 64.0)
- added R1803: 100R PWM_SER, R_0603_1608Metric, F.Cu at (236.0, 64.0)
- added R1804: 10K INA_PULLDOWN, R_0603_1608Metric, F.Cu at (240.0, 64.0)
- added R1805: 10K INB_PULLDOWN, R_0603_1608Metric, F.Cu at (244.0, 64.0)
- added R1806: 10K PWM_PULLDOWN, R_0603_1608Metric, F.Cu at (248.0, 64.0)
- added R1807: 4K7 DIAG_PULLUP, R_0603_1608Metric, F.Cu at (230.0, 68.0)
- added R1808: 10K CS_DIS_PULLDOWN, R_0603_1608Metric, F.Cu at (234.0, 68.0)
- added R1809: 1K 1% CS_LOAD, R_0603_1608Metric, F.Cu at (238.0, 68.0)
- added R1810: 10K ADC_SERIES, R_0603_1608Metric, F.Cu at (242.0, 68.0)
- added R3011: 47K SLOT_S1_ID0, R_0603_1608Metric, F.Cu at (43.0, 120.0)
- added R3012: 47K SLOT_S1_ID1, R_0603_1608Metric, F.Cu at (47.0, 120.0)
- added R3021: 0R SLOT_S2_ID0, R_0603_1608Metric, F.Cu at (103.0, 120.0)
- added R3022: 47K SLOT_S2_ID1, R_0603_1608Metric, F.Cu at (107.0, 120.0)
- added R3031: 47K SLOT_S3_ID0, R_0603_1608Metric, F.Cu at (163.0, 120.0)
- added R3032: 0R SLOT_S3_ID1, R_0603_1608Metric, F.Cu at (167.0, 120.0)
- added R3041: 0R SLOT_S4_ID0, R_0603_1608Metric, F.Cu at (205.0, 120.0)
- added R3042: 0R SLOT_S4_ID1, R_0603_1608Metric, F.Cu at (209.0, 120.0)
- moved D230 71.2 mm to (110.0, 88.0)
- moved F230 70.2 mm to (84.0, 88.0)
- moved C230 68.0 mm to (128.0, 100.0)
- moved D231 67.4 mm to (118.0, 88.0)
- moved C233 52.0 mm to (169.0, 100.0)
- moved C231 50.1 mm to (126.0, 88.0)
- moved C232 49.2 mm to (131.0, 88.0)
- moved DC1 42.9 mm to (138.0, 85.0)
- moved C234 33.3 mm to (165.0, 88.0)
- moved C235 33.3 mm to (171.0, 88.0)
- moved H2 15.0 mm to (208.0, 90.0)
Connections:
- J1 pad 1: (no net) -> FUSED_12V_CH1
- J1 pad 2: (no net) -> GND
- J10 pad 1: (no net) -> CH2_OUTA
- J10 pad 2: (no net) -> CH2_OUTB
- J11 pad 1: (no net) -> CH3_OUTA
- J11 pad 2: (no net) -> CH3_OUTB
- J12 pad 1: (no net) -> CH4_OUTA
- J12 pad 2: (no net) -> CH4_OUTB
- J13 pad 1: (no net) -> CH5_OUTA
- J13 pad 2: (no net) -> CH5_OUTB
- J14 pad 1: (no net) -> CH6_OUTA
- J14 pad 2: (no net) -> CH6_OUTB
- J15 pad 1: (no net) -> CH7_OUTA
- J15 pad 2: (no net) -> CH7_OUTB
- J16 pad 1: (no net) -> CH8_OUTA
- J16 pad 2: (no net) -> CH8_OUTB
- J2 pad 1: (no net) -> FUSED_12V_CH2
- J2 pad 2: (no net) -> GND
- J3 pad 1: (no net) -> FUSED_12V_CH3
- J3 pad 2: (no net) -> GND
- J4 pad 1: (no net) -> FUSED_12V_CH4
- J4 pad 2: (no net) -> GND
- J5 pad 1: (no net) -> FUSED_12V_CH5
- J5 pad 2: (no net) -> GND
- J6 pad 1: (no net) -> FUSED_12V_CH6
- J6 pad 2: (no net) -> GND
- J7 pad 1: (no net) -> FUSED_12V_CH7
- J7 pad 2: (no net) -> GND
- J8 pad 1: (no net) -> FUSED_12V_CH8
- J8 pad 2: (no net) -> GND
- J9 pad 1: (no net) -> CH1_OUTA
- J9 pad 2: (no net) -> CH1_OUTB
- MOD1 pad 1: (no net) -> GND
- MOD1 pad 10: (no net) -> CH2_CURRENT_ADC
- MOD1 pad 11: (no net) -> S1_3V3
- MOD1 pad 12: (no net) -> CH1_INB_MCU
- MOD1 pad 15: (no net) -> S1_SLOT_ID0
- MOD1 pad 2: (no net) -> CH1_INA_MCU
- MOD1 pad 20: (no net) -> CH1_CURRENT_ADC
- MOD1 pad 21: (no net) -> LOGIC_5V
- MOD1 pad 22: (no net) -> CH1_PWM_MCU
- MOD1 pad 26: (no net) -> CH2_INA_MCU
- MOD1 pad 27: (no net) -> CH1_DIAG
- MOD1 pad 3: (no net) -> CH2_DIAG
- MOD1 pad 31: (no net) -> GND
- MOD1 pad 32: (no net) -> CH2_PWM_MCU
- MOD1 pad 36: (no net) -> CH2_INB_MCU
- MOD1 pad 7: (no net) -> S1_SLOT_ID1
- MOD2 pad 1: (no net) -> GND
- MOD2 pad 10: (no net) -> CH4_CURRENT_ADC
- MOD2 pad 11: (no net) -> S2_3V3
- MOD2 pad 12: (no net) -> CH3_INB_MCU
- MOD2 pad 15: (no net) -> S2_SLOT_ID0
- MOD2 pad 2: (no net) -> CH3_INA_MCU
- MOD2 pad 20: (no net) -> CH3_CURRENT_ADC
- MOD2 pad 21: (no net) -> LOGIC_5V
- MOD2 pad 22: (no net) -> CH3_PWM_MCU
- MOD2 pad 26: (no net) -> CH4_INA_MCU
- MOD2 pad 27: (no net) -> CH3_DIAG
- MOD2 pad 3: (no net) -> CH4_DIAG
- MOD2 pad 31: (no net) -> GND
- MOD2 pad 32: (no net) -> CH4_PWM_MCU
- MOD2 pad 36: (no net) -> CH4_INB_MCU
- MOD2 pad 7: (no net) -> S2_SLOT_ID1
- MOD3 pad 1: (no net) -> GND
- MOD3 pad 10: (no net) -> CH6_CURRENT_ADC
- MOD3 pad 11: (no net) -> S3_3V3
- MOD3 pad 12: (no net) -> CH5_INB_MCU
- MOD3 pad 15: (no net) -> S3_SLOT_ID0
- MOD3 pad 2: (no net) -> CH5_INA_MCU
- MOD3 pad 20: (no net) -> CH5_CURRENT_ADC
- MOD3 pad 21: (no net) -> LOGIC_5V
- MOD3 pad 22: (no net) -> CH5_PWM_MCU
- MOD3 pad 26: (no net) -> CH6_INA_MCU
- MOD3 pad 27: (no net) -> CH5_DIAG
- MOD3 pad 3: (no net) -> CH6_DIAG
- MOD3 pad 31: (no net) -> GND
- MOD3 pad 32: (no net) -> CH6_PWM_MCU
- MOD3 pad 36: (no net) -> CH6_INB_MCU
- MOD3 pad 7: (no net) -> S3_SLOT_ID1
- MOD4 pad 1: (no net) -> GND
- MOD4 pad 10: (no net) -> CH8_CURRENT_ADC
- MOD4 pad 11: (no net) -> S4_3V3
- MOD4 pad 12: (no net) -> CH7_INB_MCU
- MOD4 pad 15: (no net) -> S4_SLOT_ID0
- MOD4 pad 2: (no net) -> CH7_INA_MCU
- MOD4 pad 20: (no net) -> CH7_CURRENT_ADC
- MOD4 pad 21: (no net) -> LOGIC_5V
- MOD4 pad 22: (no net) -> CH7_PWM_MCU
- MOD4 pad 26: (no net) -> CH8_INA_MCU
- MOD4 pad 27: (no net) -> CH7_DIAG
- MOD4 pad 3: (no net) -> CH8_DIAG
- MOD4 pad 31: (no net) -> GND
- MOD4 pad 32: (no net) -> CH8_PWM_MCU
- MOD4 pad 36: (no net) -> CH8_INB_MCU
- MOD4 pad 7: (no net) -> S4_SLOT_ID1
- U1 pad 1: (no net) -> CH1_OUTA
- U1 pad 10: (no net) -> CH1_INB
- U1 pad 12: (no net) -> FUSED_12V_CH1
- U1 pad 13: (no net) -> FUSED_12V_CH1
- U1 pad 15: (no net) -> CH1_OUTB
- U1 pad 16: (no net) -> CH1_OUTB
- U1 pad 18: (no net) -> GND
- U1 pad 19: (no net) -> GND
- U1 pad 20: (no net) -> GND
- U1 pad 21: (no net) -> CH1_OUTB
- U1 pad 23: (no net) -> FUSED_12V_CH1
- U1 pad 25: (no net) -> CH1_OUTA
- U1 pad 26: (no net) -> GND
- U1 pad 27: (no net) -> GND
- U1 pad 28: (no net) -> GND
- U1 pad 3: (no net) -> FUSED_12V_CH1
- U1 pad 30: (no net) -> CH1_OUTA
- U1 pad 4: (no net) -> CH1_INA
- U1 pad 5: (no net) -> CH1_DIAG
- U1 pad 6: (no net) -> CH1_CS_DIS
- U1 pad 7: (no net) -> CH1_PWM
- U1 pad 8: (no net) -> CH1_CS_RAW
- U1 pad 9: (no net) -> CH1_DIAG
- U2 pad 1: (no net) -> CH2_OUTA
- U2 pad 10: (no net) -> CH2_INB
- U2 pad 12: (no net) -> FUSED_12V_CH2
- U2 pad 13: (no net) -> FUSED_12V_CH2
- U2 pad 15: (no net) -> CH2_OUTB
- U2 pad 16: (no net) -> CH2_OUTB
- U2 pad 18: (no net) -> GND
- U2 pad 19: (no net) -> GND
- U2 pad 20: (no net) -> GND
- U2 pad 21: (no net) -> CH2_OUTB
- U2 pad 23: (no net) -> FUSED_12V_CH2
- U2 pad 25: (no net) -> CH2_OUTA
- U2 pad 26: (no net) -> GND
- U2 pad 27: (no net) -> GND
- U2 pad 28: (no net) -> GND
- U2 pad 3: (no net) -> FUSED_12V_CH2
- U2 pad 30: (no net) -> CH2_OUTA
- U2 pad 4: (no net) -> CH2_INA
- U2 pad 5: (no net) -> CH2_DIAG
- U2 pad 6: (no net) -> CH2_CS_DIS
- U2 pad 7: (no net) -> CH2_PWM
- U2 pad 8: (no net) -> CH2_CS_RAW
- U2 pad 9: (no net) -> CH2_DIAG
- U3 pad 1: (no net) -> CH3_OUTA
- U3 pad 10: (no net) -> CH3_INB
- U3 pad 12: (no net) -> FUSED_12V_CH3
- U3 pad 13: (no net) -> FUSED_12V_CH3
- U3 pad 15: (no net) -> CH3_OUTB
- U3 pad 16: (no net) -> CH3_OUTB
- U3 pad 18: (no net) -> GND
- U3 pad 19: (no net) -> GND
- U3 pad 20: (no net) -> GND
- U3 pad 21: (no net) -> CH3_OUTB
- U3 pad 23: (no net) -> FUSED_12V_CH3
- U3 pad 25: (no net) -> CH3_OUTA
- U3 pad 26: (no net) -> GND
- U3 pad 27: (no net) -> GND
- U3 pad 28: (no net) -> GND
- U3 pad 3: (no net) -> FUSED_12V_CH3
- U3 pad 30: (no net) -> CH3_OUTA
- U3 pad 4: (no net) -> CH3_INA
- U3 pad 5: (no net) -> CH3_DIAG
- U3 pad 6: (no net) -> CH3_CS_DIS
- U3 pad 7: (no net) -> CH3_PWM
- U3 pad 8: (no net) -> CH3_CS_RAW
- U3 pad 9: (no net) -> CH3_DIAG
- U4 pad 1: (no net) -> CH4_OUTA
- U4 pad 10: (no net) -> CH4_INB
- U4 pad 12: (no net) -> FUSED_12V_CH4
- U4 pad 13: (no net) -> FUSED_12V_CH4
- U4 pad 15: (no net) -> CH4_OUTB
- U4 pad 16: (no net) -> CH4_OUTB
- U4 pad 18: (no net) -> GND
- U4 pad 19: (no net) -> GND
- U4 pad 20: (no net) -> GND
- U4 pad 21: (no net) -> CH4_OUTB
- U4 pad 23: (no net) -> FUSED_12V_CH4
- U4 pad 25: (no net) -> CH4_OUTA
- U4 pad 26: (no net) -> GND
- U4 pad 27: (no net) -> GND
- U4 pad 28: (no net) -> GND
- U4 pad 3: (no net) -> FUSED_12V_CH4
- U4 pad 30: (no net) -> CH4_OUTA
- U4 pad 4: (no net) -> CH4_INA
- U4 pad 5: (no net) -> CH4_DIAG
- U4 pad 6: (no net) -> CH4_CS_DIS
- U4 pad 7: (no net) -> CH4_PWM
- U4 pad 8: (no net) -> CH4_CS_RAW
- U4 pad 9: (no net) -> CH4_DIAG
- U5 pad 1: (no net) -> CH5_OUTA
- U5 pad 10: (no net) -> CH5_INB
- U5 pad 12: (no net) -> FUSED_12V_CH5
- U5 pad 13: (no net) -> FUSED_12V_CH5
- U5 pad 15: (no net) -> CH5_OUTB
- U5 pad 16: (no net) -> CH5_OUTB
- U5 pad 18: (no net) -> GND
- U5 pad 19: (no net) -> GND
- U5 pad 20: (no net) -> GND
- U5 pad 21: (no net) -> CH5_OUTB
- U5 pad 23: (no net) -> FUSED_12V_CH5
- U5 pad 25: (no net) -> CH5_OUTA
- U5 pad 26: (no net) -> GND
- U5 pad 27: (no net) -> GND
- U5 pad 28: (no net) -> GND
- U5 pad 3: (no net) -> FUSED_12V_CH5
- U5 pad 30: (no net) -> CH5_OUTA
- U5 pad 4: (no net) -> CH5_INA
- U5 pad 5: (no net) -> CH5_DIAG
- U5 pad 6: (no net) -> CH5_CS_DIS
- U5 pad 7: (no net) -> CH5_PWM
- U5 pad 8: (no net) -> CH5_CS_RAW
- U5 pad 9: (no net) -> CH5_DIAG
- U6 pad 1: (no net) -> CH6_OUTA
- U6 pad 10: (no net) -> CH6_INB
- U6 pad 12: (no net) -> FUSED_12V_CH6
- U6 pad 13: (no net) -> FUSED_12V_CH6
- U6 pad 15: (no net) -> CH6_OUTB
- U6 pad 16: (no net) -> CH6_OUTB
- U6 pad 18: (no net) -> GND
- U6 pad 19: (no net) -> GND
- U6 pad 20: (no net) -> GND
- U6 pad 21: (no net) -> CH6_OUTB
- U6 pad 23: (no net) -> FUSED_12V_CH6
- U6 pad 25: (no net) -> CH6_OUTA
- U6 pad 26: (no net) -> GND
- U6 pad 27: (no net) -> GND
- U6 pad 28: (no net) -> GND
- U6 pad 3: (no net) -> FUSED_12V_CH6
- U6 pad 30: (no net) -> CH6_OUTA
- U6 pad 4: (no net) -> CH6_INA
- U6 pad 5: (no net) -> CH6_DIAG
- U6 pad 6: (no net) -> CH6_CS_DIS
- U6 pad 7: (no net) -> CH6_PWM
- U6 pad 8: (no net) -> CH6_CS_RAW
- U6 pad 9: (no net) -> CH6_DIAG
- U7 pad 1: (no net) -> CH7_OUTA
- U7 pad 10: (no net) -> CH7_INB
- U7 pad 12: (no net) -> FUSED_12V_CH7
- U7 pad 13: (no net) -> FUSED_12V_CH7
- U7 pad 15: (no net) -> CH7_OUTB
- U7 pad 16: (no net) -> CH7_OUTB
- U7 pad 18: (no net) -> GND
- U7 pad 19: (no net) -> GND
- U7 pad 20: (no net) -> GND
- U7 pad 21: (no net) -> CH7_OUTB
- U7 pad 23: (no net) -> FUSED_12V_CH7
- U7 pad 25: (no net) -> CH7_OUTA
- U7 pad 26: (no net) -> GND
- U7 pad 27: (no net) -> GND
- U7 pad 28: (no net) -> GND
- U7 pad 3: (no net) -> FUSED_12V_CH7
- U7 pad 30: (no net) -> CH7_OUTA
- U7 pad 4: (no net) -> CH7_INA
- U7 pad 5: (no net) -> CH7_DIAG
- U7 pad 6: (no net) -> CH7_CS_DIS
- U7 pad 7: (no net) -> CH7_PWM
- U7 pad 8: (no net) -> CH7_CS_RAW
- U7 pad 9: (no net) -> CH7_DIAG
- U8 pad 1: (no net) -> CH8_OUTA
- U8 pad 10: (no net) -> CH8_INB
- U8 pad 12: (no net) -> FUSED_12V_CH8
- U8 pad 13: (no net) -> FUSED_12V_CH8
- U8 pad 15: (no net) -> CH8_OUTB
- U8 pad 16: (no net) -> CH8_OUTB
- U8 pad 18: (no net) -> GND
- U8 pad 19: (no net) -> GND
- U8 pad 20: (no net) -> GND
- U8 pad 21: (no net) -> CH8_OUTB
- U8 pad 23: (no net) -> FUSED_12V_CH8
- U8 pad 25: (no net) -> CH8_OUTA
- U8 pad 26: (no net) -> GND
- U8 pad 27: (no net) -> GND
- U8 pad 28: (no net) -> GND
- U8 pad 3: (no net) -> FUSED_12V_CH8
- U8 pad 30: (no net) -> CH8_OUTA
- U8 pad 4: (no net) -> CH8_INA
- U8 pad 5: (no net) -> CH8_DIAG
- U8 pad 6: (no net) -> CH8_CS_DIS
- U8 pad 7: (no net) -> CH8_PWM
- U8 pad 8: (no net) -> CH8_CS_RAW
- U8 pad 9: (no net) -> CH8_DIAG
