File: hardware/DOOR-8CH/kicad/DOOR-8CH.kicad_pcb (KiCad board)
At the start: 4 copper layers, 260 x 160 mm, 230 parts, among them J1 FUSED_12V_CH1, J10 ACTUATOR_CH2, J11 ACTUATOR_CH3, J12 ACTUATOR_CH4, J13 ACTUATOR_CH5, J14 ACTUATOR_CH6, J15 ACTUATOR_CH7, J16 ACTUATOR_CH8, J2 FUSED_12V_CH2, J201 REED_A_OPEN_3V3_SIG_GND, J202 REED_A_CLOSED_3V3_SIG_GND, J203 REED_A_IN_PLACE_3V3_SIG_GND, J204 REED_B_OPEN_3V3_SIG_GND, J205 REED_B_CLOSED_3V3_SIG_GND, J206 REED_B_IN_PLACE_3V3_SIG_GND, J211 CAP_CS1_GND, J212 CAP_CS2_GND, J213 CAP_CS3_GND, J214 CAP_CS4_GND, J215 CAP_CS5_GND, J216 CAP_CS6_GND, J217 CAP_CS7_GND, J218 CAP_CS8_GND, J220 SWD_S1_3V3_DIO_CLK_NRST_GND, J230 LOGIC_12V_GND, J240 CANH_CANL_GND_SHIELD, J3 FUSED_12V_CH3, J4 FUSED_12V_CH4, J5 FUSED_12V_CH5, J6 FUSED_12V_CH6, J7 FUSED_12V_CH7, J8 FUSED_12V_CH8, J9 ACTUATOR_CH1, U1 VNH5019A-E, U2 VNH5019A-E, U230 AMS1117-3V3, U250 25LC256_SOIC8_CARRIER_ID, U3 VNH5019A-E, U4 VNH5019A-E, U5 VNH5019A-E, U6 VNH5019A-E, U7 VNH5019A-E, U8 VNH5019A-E

Commit message: Route channel 4 current ADC to STM32
Routing:
- net CH4_CURRENT_ADC: track 7.39 -> 109.5 mm, vias 0 -> 2
Changed lines of the file:
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@@
+	)
+	(segment
+		(start 115.16 126)
+		(end 115.16 130.139999)
+		(width 0.25)
+		(layer "F.Cu")
+		(net "CH4_CURRENT_ADC")
+	)
+	(segment
+		(start 120.825 68)
+		(end 124 70)
+		(width 0.25)
+		(layer "F.Cu")
+		(net "CH4_CURRENT_ADC")
+	)
+	(segment
+		(start 120.825 68)
+		(end 124 70)
+		(width 0.25)
+		(layer "F.Cu")
+		(net "CH4_CURRENT_ADC")
+	)
+	(segment
+		(start 124 105)
+		(end 128 120)
+		(width 0.25)
+		(layer "F.Cu")
+		(net "CH4_CURRENT_ADC")
 	)
 	(segment
 		(start 120.83 68)
 		(end 119.94 72)
+		(width 0.25)
+		(layer "F.Cu")
+		(net "CH4_CURRENT_ADC")
+	)
+	(segment
+		(start 120.825 68)
+		(end 124 70)
+		(width 0.25)
+		(layer "F.Cu")
+		(net "CH4_CURRENT_ADC")
+	)
+	(segment
+		(start 120.825 68)
+		(end 124 70)
+		(width 0.25)
+		(layer "F.Cu")
+		(net "CH4_CURRENT_ADC")
+	)
+	(segment
+		(start 120.825 68)
+		(end 124 70)
 		(width 0.25)
 		(layer "F.Cu")
@@
 		(net "CH4_CURRENT_ADC")
 	)
+	(segment
+		(start 128 120)
+		(end 130 126)
+		(width 0.25)
+		(layer "F.Cu")
+		(net "CH4_CURRENT_ADC")
+	)
+	(segment
+		(start 130 126)
+		(end 115.16 126)
+		(width 0.25)
+		(layer "F.Cu")
+		(net "CH4_CURRENT_ADC")
+	)
+	(segment
+		(start 120.825 68)
+		(end 124 70)
+		(width 0.25)
+		(layer "F.Cu")
+		(net "CH4_CURRENT_ADC")
+	)
+	(segment
+		(start 120.825 68)
+		(end 124 70)
+		(width 0.25)
+		(layer "F.Cu")
+		(net "CH4_CURRENT_ADC")
+	)
+	(via
+		(at 124 70)
+		(size 0.8)
+		(drill 0.35)
+		(layers "F.Cu" "B.Cu")
+		(net "CH4_CURRENT_ADC")
+	)
+	(via
+		(at 124 105)
+		(size 0.8)
+		(drill 0.35)
+		(layers "F.Cu" "B.Cu")
+		(net "CH4_CURRENT_ADC")
+	)
+	(segment
+		(start 124 70)
+		(end 124 105)
+		(width 0.25)
+		(layer "In1.Cu")
+		(net "CH4_CURRENT_ADC")
+	)
