File: hardware/DOOR-8CH/kicad/DOOR-8CH-control-can.kicad_sch (KiCad schematic)
At the start: 25 parts, among them J220 SWD_S1_3V3_DIO_CLK_NRST_GND, U250 25LC256_SOIC8_CARRIER_ID

Commit message: Add DOOR-8CH power-fail hold-up and persistent journal
Connections:
- net LOGIC_3V3: no longer R260.2 (P2), R261.2 (P2), R262.2 (P2), U250.5 (P5)
- net S1_3V3: now also R260.2 (P2), R261.2 (P2), R262.2 (P2), U250.5 (P5)
Changed lines of the file:
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@@
     (effects (font (size 0.8 0.8)))
   )
-  (global_label "LOGIC_3V3" (shape passive) (at 491.49 71.12 0)
+  (global_label "S1_3V3" (shape passive) (at 491.49 71.12 0)
     (effects (font (size 0.8 0.8)))
   )
@@
     (effects (font (size 0.8 0.8)))
   )
-  (global_label "LOGIC_3V3" (shape passive) (at 359.41 127.0 0)
+  (global_label "S1_3V3" (shape passive) (at 359.41 127.0 0)
     (effects (font (size 0.8 0.8)))
   )
@@
     (effects (font (size 0.8 0.8)))
   )
-  (global_label "LOGIC_3V3" (shape passive) (at 491.49 127.0 0)
+  (global_label "S1_3V3" (shape passive) (at 491.49 127.0 0)
     (effects (font (size 0.8 0.8)))
   )
@@
     (effects (font (size 0.8 0.8)))
   )
-  (global_label "LOGIC_3V3" (shape passive) (at 93.98 132.08 0)
+  (global_label "S1_3V3" (shape passive) (at 93.98 132.08 0)
     (effects (font (size 0.8 0.8)))
   )
@@
   )
   (symbol_instances
-    (path "/8d0ac401-ce70-49c3-97bd-c1f6c42a4fe4"
+    (path "/ef91d359-06a9-4143-9d3e-d7cd845906aa"
       (reference "ESP1") (unit 1) (value "ESP32_S3_DEVKITC_DOUBLE_DOOR_ONLY") (footprint "")
     )
-    (path "/f47fbafa-de9e-4fa5-8cd8-0329862abf09"
+    (path "/4fddec43-1447-4c77-9940-52ea7d7a61ba"
       (reference "MOD3") (unit 1) (value "STM32F103C8T6_MINI_SLOT_S3") (footprint "")
     )
-    (path "/78dfe3cb-284e-4978-857b-81b78c40b3c3"
+    (path "/36b2083d-f5c1-4442-9cdb-a6cd9372d5e6"
       (reference "MOD4") (unit 1) (value "STM32F103C8T6_MINI_SLOT_S4") (footprint "")
     )
-    (path "/78658456-1972-4548-8472-dd63d1693036"
+    (path "/a7b7cc74-b5df-4d34-b3f2-b4370c1bef0c"
       (reference "RF1") (unit 1) (value "CC1101_433MHZ") (footprint "")
     )
-    (path "/b881f627-93c6-4322-88c5-0aef42590a16"
+    (path "/1ac0860f-701a-4f99-adfc-a364723c4737"
       (reference "U250") (unit 1) (value "25LC256_SOIC8_CARRIER_ID") (footprint "")
     )
-    (path "/5afe7815-1581-4496-880f-fc9e37a6cc77"
+    (path "/fba06761-a8ed-4f86-86f9-db37c70dabf8"
       (reference "CAN1") (unit 1) (value "SN65HVD230_MASTER_CAN") (footprint "")
     )
-    (path "/2a89d058-ab98-4b41-971c-cfe1ea9736a7"
+    (path "/efe7f262-99ab-40d7-98bd-c82918515baf"
       (reference "CAN2") (unit 1) (value "SN65HVD230_ESP_CAN_OPTION") (footprint "")
     )
-    (path "/ebbb756c-685d-4566-91e1-c5f3bccf6741"
+    (path "/cfed7a9d-6b9a-4d0e-8038-9d41bde3ecb2"
       (reference "J220") (unit 1) (value "SWD_S1_3V3_DIO_CLK_NRST_GND") (footprint "")
     )
-    (path "/97e36aca-a830-4f5d-93ed-52f47da07888"
+    (path "/da2f2415-0efa-447e-865d-3a1453ec5ae9"
       (reference "R250") (unit 1) (value "100R_UART_TX") (footprint "")
     )
-    (path "/b43e3cf9-dcbf-48a2-b8aa-06bb5ee849ce"
+    (path "/aa3534cb-d1a3-470a-80ed-125b26cc02c1"
       (reference "R251") (unit 1) (value "100R_UART_TX") (footprint "")
     )
-    (path "/72d713a7-1bfa-42e1-828e-c66a3c119161"
+    (path "/9a2f2995-615e-41e9-ac83-c51c36e496c9"
       (reference "R252") (unit 1) (value "100R_UART_TX") (footprint "")
     )
-    (path "/a9e100a8-4e95-442b-a007-f8fa985f80f1"
+    (path "/cce03949-325b-4c28-a65f-74e6e9a43639"
       (reference "R253") (unit 1) (value "100R_UART_TX") (footprint "")
     )
-    (path "/fa3098ab-8a21-428d-abc8-200198ca53c2"
+    (path "/969e7553-88ac-483a-9eec-06ec02df3e70"
       (reference "R254") (unit 1) (value "100R_UART_TX") (footprint "")
     )
-    (path "/2d1287ee-3755-4037-92ad-9b8e23306e74"
+    (path "/b4661009-6c45-4bc8-b2ab-162e63a08eb5"
       (reference "R255") (unit 1) (value "100R_UART_TX") (footprint "")
     )
-    (path "/ba802406-e07f-4171-bc20-ad29decf7be8"
+    (path "/92aad20d-5fd3-450a-9eae-39f4faf996f8"
       (reference "R260") (unit 1) (value "10K_EEPROM_CS_PULLUP") (footprint "")
     )
-    (path "/f852fd98-518d-4818-884a-3b44328ac8eb"
+    (path "/6380a8e6-6f93-49bb-9612-7ff34250df43"
       (reference "R261") (unit 1) (value "10K_EEPROM_WP_PULLUP") (footprint "")
     )
-    (path "/eca12e76-5704-4e1d-bb1f-ab9d257928d6"
+    (path "/5680007a-a2a6-4b54-b325-3c6f9e32b821"
       (reference "R262") (unit 1) (value "10K_EEPROM_HOLD_PULLUP") (footprint "")
     )
-    (path "/2e1fa2ab-f0f0-4751-bc3f-73c85940858e"
+    (path "/671572e9-bfa1-437c-a24b-b10242a7ed0d"
       (reference "R3011") (unit 1) (value "47K SLOT_S1_ID0") (footprint "")
     )
-    (path "/4898aef7-f5ea-4773-9936-a06499d79595"
+    (path "/2b933740-102c-4f8e-ad5f-46b3dcfa9c65"
       (reference "R3012") (unit 1) (value "47K SLOT_S1_ID1") (footprint "")
     )
-    (path "/1333fb20-fa0a-48ec-9331-f6578b5e6476"
+    (path "/a09d9990-2d02-428f-992b-43c45e1ae329"
       (reference "R3021") (unit 1) (value "0R SLOT_S2_ID0") (footprint "")
     )
-    (path "/77ac29a6-8129-4b80-b11b-88192a9123ae"
+    (path "/378c55d9-0956-4d0d-9438-67f393f78205"
       (reference "R3022") (unit 1) (value "47K SLOT_S2_ID1") (footprint "")
     )
-    (path "/18d5a885-a663-4896-b925-553880510561"
+    (path "/31e9eefe-539b-4fa2-bb13-e24fc961bc2c"
       (reference "R3031") (unit 1) (value "47K SLOT_S3_ID0") (footprint "")
     )
-    (path "/40fd946f-1cb1-4dc5-b43d-d8b91dbc1760"
+    (path "/927a78bf-0f68-45a9-af00-ed7e98614a0f"
       (reference "R3032") (unit 1) (value "0R SLOT_S3_ID1") (footprint "")
     )
-    (path "/9e7602e9-b096-4aac-b1e9-ffdc10067bc8"
+    (path "/de197164-e386-4993-af83-7b18fa4b33aa"
       (reference "R3041") (unit 1) (value "0R SLOT_S4_ID0") (footprint "")
     )
-    (path "/952887e4-1f71-4123-ad6c-00a8a5d4a5b2"
+    (path "/d39bf28f-7f86-4a00-9e40-305398d30987"
       (reference "R3042") (unit 1) (value "0R SLOT_S4_ID1") (footprint "")
     )
