File: hardware/DOOR-8CH/kicad/DOOR-8CH-other.kicad_sch (KiCad schematic)
At the start: 25 parts, among them J240 CANH_CANL_GND_SHIELD

Commit message: Add DOOR-8CH power-fail hold-up and persistent journal
Parts:
- added C271: 100NF_PGOOD_FILTER, symbol DOOR8CH:GEN_P1_P2
- added C280: 4700UF_10V_LOW_ESR_S1_HOLDUP, symbol DOOR8CH:GEN_P1_P2
- added R271: 10K_1%_PGOOD_BOTTOM, symbol DOOR8CH:GEN_P1_P2
Connections:
- net GND: now also C271.2 (P2), C280.2 (P2), R271.2 (P2)
- new net PGOOD_SENSE: C271.1 (P1), R271.1 (P1)
- new net S1_5V_HOLD: C280.1 (P1)
