File: hardware/DOOR-8CH/kicad/DOOR-8CH-power.kicad_sch (KiCad schematic)
At the start: 19 parts, among them J230 LOGIC_12V_GND, U230 AMS1117-3V3

Commit message: Add DOOR-8CH power-fail hold-up and persistent journal
Parts:
- added C270: 100NF_25V_PGOOD_VDD, symbol DOOR8CH:GEN_P1_P2
- added D280: SS34_S1_HOLDUP_ISOLATION, symbol DOOR8CH:GEN_P1_P2
- added R270: 226K_1%_PGOOD_TOP, symbol DOOR8CH:GEN_P1_P2
- added R272: 10K_PGOOD_PULLUP, symbol DOOR8CH:GEN_P1_P2
- added U270: TLV6700DDCR_POWER_MONITOR, symbol DOOR8CH:GEN_P1_P2_P3_P4_P5_P6
Connections:
- net GND: now also C270.2 (P2), U270.2 (P2), U270.6 (P6)
- net LOGIC_12V_FUSED: now also C270.1 (P1), R270.1 (P1), U270.5 (P5)
- net LOGIC_3V3: no longer C250.1 (P1)
- net LOGIC_5V: now also D280.2 (P2)
- net S1_3V3: now also C250.1 (P1), R272.1 (P1)
- new net PGOOD_SENSE: R270.2 (P2), U270.1 (P1)
- new net POWER_GOOD: R272.2 (P2), U270.3 (P3), U270.4 (P4)
- new net S1_5V_HOLD: D280.1 (P1)
