File: hardware/DOOR-8CH/kicad/DOOR-8CH-reeds.kicad_sch (KiCad schematic)
At the start: 8 parts, among them J201 REED_A_OPEN_3V3_SIG_GND, J202 REED_A_CLOSED_3V3_SIG_GND, J203 REED_A_IN_PLACE_3V3_SIG_GND, J204 REED_B_OPEN_3V3_SIG_GND, J205 REED_B_CLOSED_3V3_SIG_GND, J206 REED_B_IN_PLACE_3V3_SIG_GND

Commit message: Add DOOR-8CH power-fail hold-up and persistent journal
Connections:
- net LOGIC_5V: no longer MOD1.40 (P40)
- net POWER_GOOD: now reaches MOD1.31 (P31)
- new net S1_5V_HOLD: MOD1.40 (P40)
- no-connect marks 23 -> 22
Changed lines of the file:
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@@
   (paper "A2")
   (no_connect (at 93.98 49.53))
-  (no_connect (at 93.98 67.31))
   (no_connect (at 93.98 90.17))
   (no_connect (at 93.98 92.71))
@@
     (effects (font (size 0.8 0.8)))
   )
-  (global_label "LOGIC_5V" (shape passive) (at 93.98 44.45 0)
+  (global_label "S1_5V_HOLD" (shape passive) (at 93.98 44.45 0)
     (effects (font (size 0.8 0.8)))
   )
@@
   )
   (global_label "CAP_RESET" (shape passive) (at 93.98 64.77 0)
+    (effects (font (size 0.8 0.8)))
+  )
+  (global_label "POWER_GOOD" (shape passive) (at 93.98 67.31 0)
     (effects (font (size 0.8 0.8)))
   )
@@
   )
   (symbol_instances
-    (path "/0eb065b9-7774-457c-b421-510665d34905"
+    (path "/cee17c11-1d61-4c34-bdb9-81e669fbf13a"
       (reference "MOD1") (unit 1) (value "STM32F103C8T6_MINI_SLOT_S1") (footprint "")
     )
-    (path "/fe22ccec-52e1-433a-87ef-1d655f7ecd93"
+    (path "/e4abffaf-bf4d-4e92-a363-455cd47e06a6"
       (reference "MOD2") (unit 1) (value "STM32F103C8T6_MINI_SLOT_S2") (footprint "")
     )
-    (path "/f4658a1f-dd63-4932-b5a0-a72d2866b294"
+    (path "/6db751d8-9e77-4ed2-a1cb-49719a333385"
       (reference "J201") (unit 1) (value "REED_A_OPEN_3V3_SIG_GND") (footprint "")
     )
-    (path "/d30a0366-7cf8-40da-94a3-97f8329224ce"
+    (path "/4a345e9a-4b96-4ebd-b4cf-c8d6a92d022c"
       (reference "J202") (unit 1) (value "REED_A_CLOSED_3V3_SIG_GND") (footprint "")
     )
-    (path "/52dd540f-2ad5-4d34-bca4-58f9361536c0"
+    (path "/b8e9750d-0e54-4cef-a4cd-96f4fe7fe9f3"
       (reference "J203") (unit 1) (value "REED_A_IN_PLACE_3V3_SIG_GND") (footprint "")
     )
-    (path "/395662c6-1b22-4988-b819-c0da56299f8a"
+    (path "/1032a2b8-4b62-44c7-a5f5-8c719df12650"
       (reference "J204") (unit 1) (value "REED_B_OPEN_3V3_SIG_GND") (footprint "")
     )
-    (path "/9d836379-b25b-4273-83e5-74228ac5d36d"
+    (path "/5edbb76f-817a-4541-94c6-41960cf6770c"
       (reference "J205") (unit 1) (value "REED_B_CLOSED_3V3_SIG_GND") (footprint "")
     )
-    (path "/1acf02df-1b62-41b4-a391-c041a824c2f7"
+    (path "/0c6baf24-3a8d-45b8-92d8-2293d09ab130"
       (reference "J206") (unit 1) (value "REED_B_IN_PLACE_3V3_SIG_GND") (footprint "")
     )
