File: hardware/DOOR-8CH/kicad/DOOR-8CH.kicad_sch (KiCad schematic)
At the start: 230 parts, among them J1 FUSED_12V_CH1, J10 ACTUATOR_CH2, J11 ACTUATOR_CH3, J12 ACTUATOR_CH4, J13 ACTUATOR_CH5, J14 ACTUATOR_CH6, J15 ACTUATOR_CH7, J16 ACTUATOR_CH8, J2 FUSED_12V_CH2, J201 REED_A_OPEN_3V3_SIG_GND, J202 REED_A_CLOSED_3V3_SIG_GND, J203 REED_A_IN_PLACE_3V3_SIG_GND, J204 REED_B_OPEN_3V3_SIG_GND, J205 REED_B_CLOSED_3V3_SIG_GND, J206 REED_B_IN_PLACE_3V3_SIG_GND, J211 CAP_CS1_GND, J212 CAP_CS2_GND, J213 CAP_CS3_GND, J214 CAP_CS4_GND, J215 CAP_CS5_GND, J216 CAP_CS6_GND, J217 CAP_CS7_GND, J218 CAP_CS8_GND, J220 SWD_S1_3V3_DIO_CLK_NRST_GND, J230 LOGIC_12V_GND, J240 CANH_CANL_GND_SHIELD, J3 FUSED_12V_CH3, J4 FUSED_12V_CH4, J5 FUSED_12V_CH5, J6 FUSED_12V_CH6, J7 FUSED_12V_CH7, J8 FUSED_12V_CH8, J9 ACTUATOR_CH1, U1 VNH5019A-E, U2 VNH5019A-E, U230 AMS1117-3V3, U250 25LC256_SOIC8_CARRIER_ID, U3 VNH5019A-E, U4 VNH5019A-E, U5 VNH5019A-E, U6 VNH5019A-E, U7 VNH5019A-E, U8 VNH5019A-E

Commit message: Add DOOR-8CH power-fail hold-up and persistent journal
Parts:
- added C270: 100NF_25V_PGOOD_VDD, symbol DOOR8CH:GEN_P1_P2
- added C271: 100NF_PGOOD_FILTER, symbol DOOR8CH:GEN_P1_P2
- added C280: 4700UF_10V_LOW_ESR_S1_HOLDUP, symbol DOOR8CH:GEN_P1_P2
- added D280: SS34_S1_HOLDUP_ISOLATION, symbol DOOR8CH:GEN_P1_P2
- added R270: 226K_1%_PGOOD_TOP, symbol DOOR8CH:GEN_P1_P2
- added R271: 10K_1%_PGOOD_BOTTOM, symbol DOOR8CH:GEN_P1_P2
- added R272: 10K_PGOOD_PULLUP, symbol DOOR8CH:GEN_P1_P2
- added U270: TLV6700DDCR_POWER_MONITOR, symbol DOOR8CH:GEN_P1_P2_P3_P4_P5_P6
Connections:
- net GND: now also C270.2 (P2), C271.2 (P2), C280.2 (P2), R271.2 (P2), U270.2 (P2), U270.6 (P6)
- net LOGIC_12V_FUSED: now also C270.1 (P1), R270.1 (P1), U270.5 (P5)
- net LOGIC_3V3: no longer C250.1 (P1), R260.2 (P2), R261.2 (P2), R262.2 (P2), U250.5 (P5)
- net LOGIC_5V: now also D280.2 (P2); no longer MOD1.40 (P40)
- net S1_3V3: now also C250.1 (P1), R260.2 (P2), R261.2 (P2), R262.2 (P2), U250.5 (P5), R272.1 (P1)
- net POWER_GOOD: now reaches MOD1.31 (P31)
- net POWER_GOOD: now also R272.2 (P2), U270.3 (P3), U270.4 (P4)
- new net PGOOD_SENSE: C271.1 (P1), R270.2 (P2), R271.1 (P1), U270.1 (P1)
- new net S1_5V_HOLD: C280.1 (P1), D280.1 (P1), MOD1.40 (P40)
- no-connect marks 163 -> 162
