File: hardware/UNIVERSAL-2CH-F103-IC/kicad/UNIVERSAL-2CH-F103-IC.kicad_pcb (KiCad board)
At the start: 2 copper layers, 83 x 100 mm, 103 parts, among them J1 ACTUATOR_CH1_4P, J2 ACTUATOR_CH2_4P, J201 REED_A_OPEN_3V3_SIG_GND, J202 REED_A_CLOSED_3V3_SIG_GND, J211 CAP_CS1_GND, J212 CAP_CS2_GND, J213 CAP_CS3_GND, J220 SWD_S1_3V3_DIO_CLK_NRST_GND, J230 LOGIC_12V_GND, J240 CANH_CANL_GND_SHIELD, J280B WIRE_FROM_C280_POS, U1 VNH5019A-E, U2 VNH5019A-E, U230 AMS1117-3V3, U250 25LC256_SOIC8_CARRIER_ID, U270 TLV6700DDCR_POWER_MONITOR, U300 STM32F103C8T6, Y300 8MHz

Commit message: hardware: protect 2ch reed inputs at 5V
Parts:
- added R290: 4.7K 1% REED INPUT SERIES, R_0603_1608Metric, F.Cu at (80.0, 17.0)
- added R291: 4.7K 1% REED INPUT SERIES, R_0603_1608Metric, F.Cu at (84.0, 43.0)
- added TP290: CAP1188_3V3_WIRE_POINT, TestPoint_Pad_D1.0mm, B.Cu at (83.6, 55.4)
- J201: value REED_A_OPEN_3V3_SIG_GND -> REED_OPEN_5V_SIG_GND_PROTECTED
- J202: value REED_A_CLOSED_3V3_SIG_GND -> REED_CLOSED_5V_SIG_GND_PROTECTED
Connections:
- C250 pad 1: S1_3V3 -> S1_3V3_REED_BRANCH
- C3004 pad 1: S1_3V3 -> S1_3V3_REED_BRANCH
- C3005 pad 1: S1_3V3 -> S1_3V3_REED_BRANCH
- C3006 pad 1: S1_3V3 -> S1_3V3_REED_BRANCH
- C3007 pad 1: S1_3V3 -> S1_3V3_REED_BRANCH
- C3008 pad 1: S1_3V3 -> S1_3V3_REED_BRANCH
- C340 pad 1: S1_3V3 -> S1_3V3_REED_BRANCH
- C341 pad 1: S1_3V3 -> S1_3V3_REED_BRANCH
- D1101 pad 2: S1_3V3 -> S1_3V3_REED_BRANCH
- D1201 pad 2: S1_3V3 -> S1_3V3_REED_BRANCH
- J201 pad 1: S1_3V3 -> LOGIC_5V
- J201 pad 2: REED_A_OPEN -> REED_A_OPEN_RAW_5V
- J202 pad 1: S1_3V3 -> LOGIC_5V
- J202 pad 2: REED_A_CLOSED -> REED_A_CLOSED_RAW_5V
- J220 pad 1: S1_3V3 -> S1_3V3_REED_BRANCH
- R1107 pad 2: S1_3V3 -> S1_3V3_REED_BRANCH
- R1207 pad 2: S1_3V3 -> S1_3V3_REED_BRANCH
- R210 pad 2: S1_3V3 -> S1_3V3_REED_BRANCH
- R2301 pad 2: S1_3V3 -> S1_3V3_REED_BRANCH
- R260 pad 2: S1_3V3 -> S1_3V3_REED_BRANCH
- R261 pad 2: S1_3V3 -> S1_3V3_REED_BRANCH
- R262 pad 2: S1_3V3 -> S1_3V3_REED_BRANCH
- R272 pad 1: S1_3V3 -> S1_3V3_REED_BRANCH
- R3001 pad 1: S1_3V3 -> S1_3V3_REED_BRANCH
- U250 pad 8: S1_3V3 -> S1_3V3_REED_BRANCH
- U300 pad 1: S1_3V3 -> S1_3V3_REED_BRANCH
- U300 pad 24: S1_3V3 -> S1_3V3_REED_BRANCH
- U300 pad 36: S1_3V3 -> S1_3V3_REED_BRANCH
- U300 pad 48: S1_3V3 -> S1_3V3_REED_BRANCH
- U300 pad 9: S1_3V3 -> S1_3V3_REED_BRANCH
Routing:
- net S1_3V3: track 224.8 -> 5.63 mm, vias 4 -> 0
- net S1_3V3_REED_BRANCH: track 0.00 -> 170.2 mm, vias 0 -> 3
- net LOGIC_5V: track 70.8 -> 147.0 mm, vias 0 -> 4
- net REED_A_CLOSED_RAW_5V: track 0.00 -> 19.8 mm
- net REED_A_OPEN: track 75.1 -> 90.1 mm, vias 2 -> 3
- net REED_A_OPEN_RAW_5V: track 0.00 -> 13.2 mm
- net REED_A_CLOSED: track 74.8 -> 77.3 mm, vias 2 -> 3
Other:
- board text added: "5V SIG GND"
- board text added: "D-M9N / P-SAFE"
- board text added: "WIRE TP290 -> JP290"

Commit message: Fix 2-channel DC-DC footprint for 15x9 mm pins
Parts:
- DC1: value MP1584_FIXED_5V -> DCE001_FIXED_5V_18x13mm
- moved C237 6.32 mm to (64.0, 84.0)
Routing:
- net LOGIC_5V: track 147.0 -> 156.9 mm, vias 4 -> 6
- net GND: track 692.6 -> 699.3 mm, vias 4 -> 7
- net CAP_RESET: track 70.0 -> 74.6 mm
- net S1_3V3_REED_BRANCH: track 170.2 -> 173.8 mm
- net LOGIC_12V_PROTECTED: track 98.8 -> 97.6 mm

Commit message: Fix two-channel safety checks and protected supervisor supply
Parts:
- C340: moved to F.Cu
- moved C340 8.78 mm to (83.5, 54.8), turned to 90 degrees
Connections:
- C270 pad 1: LOGIC_12V_FUSED -> POWER_MONITOR_12V
- C340 pad 1: S1_3V3_REED_BRANCH -> S1_3V3
- R270 pad 1: LOGIC_12V_FUSED -> POWER_MONITOR_12V
- U270 pad 5: LOGIC_12V_FUSED -> POWER_MONITOR_12V
Routing:
- net LOGIC_12V_FUSED: track 59.7 -> 27.5 mm, vias 1 -> 0
- net POWER_MONITOR_12V: track 0.00 -> 10.1 mm
- net S1_3V3_REED_BRANCH: track 173.8 -> 172.6 mm
- net GND: track 699.3 -> 699.0 mm, vias 7 -> 8
- net S1_3V3: track 5.63 -> 5.86 mm, vias 0 -> 1
